File: PCD's/CanSat_2026/_autosave-CanSat_2026.kicad_sch (KiCad schematic)
At the start: 12 parts, among them J1 Conn_01x02_Pin, J2 RADIO, J3 BMP280, J4 9DOF, J5 GPS, U1 LM1085-3.3, U3 ESP32-WROOM-32D, U4 SN74AVC4T245PW, U5 NCP163ASN180T1G

Commit message: PCB
Parts:
- removed J2: RADIO, Connector_JST:JST_SH_BM06B-SRSS-TB_1x06-1MP_P1.00mm_Vertical, symbol Connector_Generic:Conn_01x06
- U5: footprint Package_TO_SOT_SMD:SOT-23-5 -> Package_SO:TSOP-5_1.65x3.05mm_P0.95mm
Changed lines of the file:
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@@
 			)
 		)
-		(property "Footprint" "Package_TO_SOT_SMD:SOT-23-5"
+		(property "Footprint" "Package_SO:TSOP-5_1.65x3.05mm_P0.95mm"
 			(at 71.12 146.05 0)
 			(effects
@@
 					(unit 1)
 				)
-			)
-		)
-	)
-	(symbol
-		(lib_id "Connector_Generic:Conn_01x06")
-		(at 177.8 135.89 270)
-		(unit 1)
-		(exclude_from_sim no)
-		(in_bom yes)
-		(on_board yes)
-		(dnp no)
-		(property "Reference" "J2"
-			(at 163.83 135.89 0)
-			(effects
-				(font
-					(size 1.27 1.27)
-				)
-			)
-		)
-		(property "Value" "RADIO"
-			(at 166.37 135.89 0)
-			(effects
-				(font
-					(size 1.27 1.27)
-				)
-			)
-		)
-		(property "Footprint" "Connector_JST:JST_SH_BM06B-SRSS-TB_1x06-1MP_P1.00mm_Vertical"
-			(at 177.8 135.89 0)
-			(effects
-				(font
-					(size 1.27 1.27)
-				)
-				(hide yes)
-			)
-		)
-		(property "Datasheet" "~"
-			(at 177.8 135.89 0)
-			(effects
-				(font
-					(size 1.27 1.27)
-				)
-				(hide yes)
-			)
-		)
-		(property "Description" "Generic connector, single row, 01x06, script generated (kicad-library-utils/schlib/autogen/connector/)"
-			(at 177.8 135.89 0)
-			(effects
-				(font
-					(size 1.27 1.27)
-				)
-				(hide yes)
-			)
-		)
-		(pin "2"
-		)
-		(pin "1"
-		)
-		(pin "4"
-		)
-		(pin "5"
-		)
-		(pin "3"
-		)
-		(pin "6"
-		)
-		(instances
-			(project ""
-				(path "/9af06756-81cc-4295-8d37-80e0f168a4af"
-					(reference "J2")
-					(unit 1)
-				)
