File: PCD's/CanSat_2026/CanSat_2026.kicad_pcb (KiCad board)
At the start: 2 copper layers, 66 x 66 mm, 9 parts, among them J1 Conn_01x02_Pin, J2 Conn_01x06, J3 Conn_01x06, J4 9DOF, J5 Conn_01x03_Pin, U1 LM1085-3.3, U2 LP5907MFX-1.8, U3 ESP32-WROOM-32D, U4 SN74AVC4T245PW

Commit message: update PCB
Parts:
- moved J2 4.61 mm to (211.5, 64.5), turned to 0 degrees
Routing:
- net Net-(J2-Pin_5): track 12.7 -> 23.4 mm
- net Net-(J2-Pin_4): track 13.3 -> 21.8 mm
- net +3.3V: track 64.2 -> 66.2 mm
- net GND: track 232.1 -> 230.3 mm
- net Net-(J3-Pin_4): track 114.1 -> 115.1 mm
- net Net-(J5-Pin_3): track 12.4 -> 13.1 mm

Commit message: update to pcb
Routing:
- net Net-(J3-Pin_4): track 115.1 -> 116.1 mm
Other:
- board text added: "GigaBebras"
- board text added: "PLS WORK"
Changed lines of the file:
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@@
 		(layer "Edge.Cuts")
+	)
+	(gr_text "GigaBebras"
+		(at 166.5 81.5 90)
+		(layer "F.Cu")
+		(effects
+			(font
+				(size 3 3)
+				(thickness 0.75)
+				(bold yes)
+			)
+			(justify left bottom)
+		)
+	)
+	(gr_text "PLS WORK"
+		(at 167 58 90)
+		(layer "B.Cu")
+		(effects
+			(font
+				(size 3 3)
+				(thickness 0.6)
+				(bold yes)
+			)
+			(justify left bottom mirror)
+		)
 	)
 	(segment
@@
 	)
 	(segment
+		(start 195.225 81.775)
+		(end 195.225 71.55)
+		(width 0.5)
+		(layer "F.Cu")
+		(net 3)
+	)
+	(segment
 		(start 182.2225 82.69)
 		(end 182.9125 82)
 		(width 0.5)
+		(layer "F.Cu")
+		(net 3)
+	)
+	(segment
+		(start 189.5 71.55)
+		(end 189.025 72.025)
+		(width 0.4)
 		(layer "F.Cu")
 		(net 3)
@@
 	)
 	(segment
+		(start 188.5 85)
+		(end 192 85)
+		(width 0.5)
+		(layer "F.Cu")
+		(net 3)
+	)
+	(segment
 		(start 179.5 64.5)
 		(end 181 63)
@@
 	)
 	(segment
-		(start 188.34 73.16)
-		(end 189.5 72)
-		(width 0.7)
-		(layer "F.Cu")
-		(net 3)
-	)
-	(segment
 		(start 195.225 67.65)
 		(end 195.225 68.3)
@@
 	)
 	(segment
-		(start 182.3775 73.16)
-		(end 188.34 73.16)
-		(width 0.7)
-		(layer "F.Cu")
-		(net 3)
-	)
-	(segment
 		(start 188.65 82)
 		(end 187.5 82)
@@
 	)
 	(segment
-		(start 186.5 83)
-		(end 188 84.5)
-		(width 0.5)
+		(start 188 73.05)
+		(end 188 73.16)
+		(width 0.2)
 		(layer "F.Cu")
 		(net 3)
@@
 	)
 	(segment
-		(start 189.5 72)
-		(end 189.5 71.55)
-		(width 0.4)
-		(layer "F.Cu")
-		(net 3)
-	)
-	(segment
-		(start 195.225 81.775)
-		(end 195.225 71.55)
-		(width 0.5)
-		(layer "F.Cu")
-		(net 3)
-	)
-	(segment
-		(start 186.5 82.5)
-		(end 186.5 83)
-		(width 0.5)
-		(layer "F.Cu")
-		(net 3)
-	)
-	(segment
-		(start 192.5 84.5)
-		(end 195.225 81.775)
-		(width 0.5)
+		(start 189.025 72.025)
+		(end 188 73.05)
+		(width 0.6)
 		(layer "F.Cu")
 		(net 3)
@@
 		(start 179.5 73.16)
 		(end 182.3775 73.16)
-		(width 1)
+		(width 0.8)
 		(layer "F.Cu")
 		(net 3)
@@
 	)
 	(segment
+		(start 186.5 83)
+		(end 188.5 85)
+		(width 0.5)
+		(layer "F.Cu")
+		(net 3)
+	)
+	(segment
 		(start 178.5 89)
 		(end 179 88.5)
@@
 		(end 186 82)
 		(width 0.5)
+		(layer "F.Cu")
+		(net 3)
+	)
+	(segment
+		(start 182.3775 73.16)
+		(end 188 73.16)
+		(width 0.6)
 		(layer "F.Cu")
 		(net 3)
@@
 	)
 	(segment
-		(start 188 84.5)
-		(end 192.5 84.5)
+		(start 192 85)
+		(end 195.225 81.775)
+		(width 0.5)
+		(layer "F.Cu")
+		(net 3)
+	)
+	(segment
+		(start 186.5 82.5)
+		(end 186.5 83)
 		(width 0.5)
 		(layer "F.Cu")
@@
 	)
 	(segment
+		(start 182.4925 85.5)
+		(end 182.2225 85.23)
+		(width 0.5)
+		(layer "F.Cu")
+		(net 9)
+	)
+	(segment
 		(start 203 47.5)
 		(end 198.5 47.5)
@@
 	)
 	(segment
-		(start 196.2635 82.7365)
-		(end 193.77 85.23)
+		(start 192.5 86.5)
+		(end 185.5 86.5)
 		(width 0.5)
 		(layer "F.Cu")
@@
 		(start 197.25 61.25)
 		(end 197.5 61.5)
+		(width 0.5)
+		(layer "F.Cu")
+		(net 9)
+	)
+	(segment
+		(start 196.5 72.5)
+		(end 196.2635 72.7365)
 		(width 0.5)
 		(layer "F.Cu")
@@
 	)
 	(segment
-		(start 196.5 72.5)
-		(end 196.2635 72.7365)
+		(start 196.5 71)
+		(end 196.5 72.5)
 		(width 0.5)
 		(layer "F.Cu")
@@
 	)
 	(segment
+		(start 185.5 86.5)
+		(end 184.5 85.5)
+		(width 0.5)
+		(layer "F.Cu")
+		(net 9)
+	)
+	(segment
 		(start 180 96)
 		(end 180 87.4525)
@@
 	)
 	(segment
+		(start 196.2635 72.7365)
+		(end 196.2635 82.7365)
+		(width 0.5)
+		(layer "F.Cu")
+		(net 9)
+	)
+	(segment
 		(start 197.5 61.5)
 		(end 199 63)
@@
 	)
 	(segment
+		(start 196.2635 82.7365)
+		(end 192.5 86.5)
+		(width 0.5)
+		(layer "F.Cu")
+		(net 9)
+	)
+	(segment
+		(start 184.5 85.5)
+		(end 182.4925 85.5)
+		(width 0.5)
+		(layer "F.Cu")
+		(net 9)
+	)
+	(segment
 		(start 180 87.4525)
-		(end 182.2225 85.23)
-		(width 0.5)
-		(layer "F.Cu")
-		(net 9)
-	)
-	(segment
-		(start 196.5 72.5)
-		(end 196.5 71)
-		(width 0.5)
-		(layer "F.Cu")
-		(net 9)
-	)
-	(segment
-		(start 196.2635 72.7365)
-		(end 196.2635 82.7365)
-		(width 0.5)
-		(layer "F.Cu")
-		(net 9)
-	)
-	(segment
-		(start 193.77 85.23)
 		(end 182.2225 85.23)
 		(width 0.5)
@@
 	)
 	(segment
+		(start 186 68)
+		(end 188.25 70.25)
+		(width 0.4)
+		(layer "F.Cu")
+		(net 23)
+	)
+	(segment
+		(start 182.4575 68)
+		(end 186 68)
+		(width 0.4)
+		(layer "F.Cu")
+		(net 23)
+	)
+	(segment
 		(start 188.25 70.25)
 		(end 189.5 70.25)
@@
 	)
 	(segment
-		(start 187 69)
-		(end 188.25 70.25)
-		(width 0.4)
-		(layer "F.Cu")
-		(net 23)
-	)
-	(segment
 		(start 182.3775 68.08)
 		(end 182.4575 68)
 		(width 0.4)
 		(layer "F.Cu")
-		(net 23)
-	)
-	(segment
-		(start 186 69)
-		(end 187 69)
-		(width 0.4)
-		(layer "F.Cu")
-		(net 23)
-	)
-	(segment
-		(start 182.4575 68)
-		(end 185 68)
-		(width 0.4)
-		(layer "F.Cu")
-		(net 23)
-	)
-	(segment
-		(start 185 68)
-		(end 186 69)
-		(width 0.4)
-		(layer "F.Cu")

Commit message: PCB
Parts:
- removed U2: LP5907MFX-1.8, Package_TO_SOT_SMD:SOT-23-5_HandSoldering
- added C1: 1uF_50V, Capacitor_THT:C_Disc_D5.0mm_W2.5mm_P5.00mm, F.Cu at (173.0, 48.0)
- added C3: 10uF_50V, Capacitor_THT:C_Radial_D6.3mm_H11.0mm_P2.50mm, F.Cu at (215.2, 80.5)
- added C4: 10uF_50V, Capacitor_THT:C_Radial_D6.3mm_H11.0mm_P2.50mm, F.Cu at (211.2, 86.5)
- added U5: NCP163ASN180T1G, Package_SO:TSOP-5_1.65x3.05mm_P0.95mm, F.Cu at (189.1, 79.1)
- J2: value Conn_01x06 -> RADIO; footprint Connector_JST:JST_GH_SM06B-GHS-TB_1x06-1MP_P1.25mm_Horizontal -> Connector_JST:JST_SH_BM06B-SRSS-TB_1x06-1MP_P1.00mm_Vertical
- J3: value Conn_01x06 -> BMP280
- J5: value Conn_01x03_Pin -> GPS
- U1: footprint Package_TO_SOT_THT:TO-220-3_Horizontal_TabUp -> Package_TO_SOT_THT:TO-220-3_Vertical
- moved J2 0.71 mm to (211.0, 64.0)
Routing:
- net GND: track 230.5 -> 285.3 mm
- net +1V8: track 24.8 -> 57.8 mm
- net +5V: track 29.9 -> 44.4 mm
- net +3.3V: track 66.2 -> 77.8 mm
- net Net-(J2-Pin_5): track 23.4 -> 19.8 mm
- net Net-(J2-Pin_4): track 21.8 -> 18.3 mm
- net Net-(J3-Pin_3): track 84.3 -> 87.0 mm
- net Net-(J3-Pin_4): track 116.1 -> 118.7 mm

Commit message: PCB updates
Parts:
- J2: value RADIO -> Conn_01x04_Pin; footprint Connector_JST:JST_SH_BM06B-SRSS-TB_1x06-1MP_P1.00mm_Vertical -> Connector_PinHeader_2.54mm:PinHeader_1x04_P2.54mm_Vertical; moved to F.Cu
- moved U1 5.73 mm to (205.0, 75.0)
- moved J2 4.78 mm to (215.5, 65.5), turned to -90 degrees
- moved J5 0.46 mm to (211.5, 53.0)
Connections:
- J2 pad 1: GND -> +5V
- J2 pad 2: unconnected-(J2-Pin_2-Pad2) -> Net-(J2-Pin_2)
- J2 pad 3: unconnected-(J2-Pin_3-Pad3) -> Net-(J2-Pin_3)
- J2 pad 4: Net-(J2-Pin_4) -> GND
- U3 pad 29: Net-(J2-Pin_4) -> Net-(J2-Pin_3)
- U3 pad 30: Net-(J2-Pin_5) -> Net-(J2-Pin_2)
- U4 pad 11: Net-(J3-Pin_3) -> unconnected-(U4-2B1-Pad11)
- U4 pad 12: unconnected-(U4-1B2-Pad12) -> Net-(J3-Pin_3)
- U4 pad 5: unconnected-(U4-1A2-Pad5) -> Net-(J4-Pin_4)
- U4 pad 6: Net-(J4-Pin_4) -> unconnected-(U4-2A1-Pad6)
Routing:
- net GND: track 285.3 -> 225.7 mm, vias 0 -> 4
- net Net-(J2-Pin_5): track 19.8 -> 0.00 mm
- net Net-(J2-Pin_2): track 0.00 -> 19.2 mm
- net Net-(J2-Pin_4): track 18.3 -> 0.00 mm
- net Net-(J2-Pin_3): track 0.00 -> 15.5 mm
- net +5V: track 44.4 -> 39.0 mm
- net +3.3V: track 77.8 -> 73.5 mm
- net Net-(J3-Pin_3): track 87.0 -> 90.7 mm
- net Net-(J3-Pin_4): track 118.7 -> 120.5 mm
- net +1V8: track 57.8 -> 58.5 mm
Other:
- board text removed: "GigaBebras"
- board text removed: "PLS WORK"
