File: PCD's/CanSat_2026/CanSat_2026.kicad_sch (KiCad schematic)
At the start: 12 parts, among them J1 Conn_01x02_Pin, J2 RADIO, J3 BMP280, J4 9DOF, J5 GPS, U1 LM1085-3.3, U3 ESP32-WROOM-32D, U4 SN74AVC4T245PW, U5 NCP163ASN180T1G

Commit message: PCB updates
Parts:
- removed J2: RADIO, Connector_JST:JST_SH_BM06B-SRSS-TB_1x06-1MP_P1.00mm_Vertical, symbol Connector_Generic:Conn_01x06
- added J2: Conn_01x04_Pin, Connector_PinHeader_2.54mm:PinHeader_1x04_P2.54mm_Vertical, symbol Connector:Conn_01x04_Pin
- U5: footprint Package_TO_SOT_SMD:SOT-23-5 -> Package_SO:TSOP-5_1.65x3.05mm_P0.95mm
Connections:
- net +5V: now also J2.1 (Pin_1)
- net GND: now also J2.4 (Pin_4)
- net at J3.3 (Pin_3), U3.33 (IO21): now also U4.12 (1B2); no longer U4.11 (2B1)
- net at U4.5 (1A2): now also J4.4 (Pin_4)
- net at U4.6 (2A1): no longer J4.4 (Pin_4)
- net at U3.29 (IO5): now also J2.3 (Pin_3)
- net at U3.30 (IO18): now also J2.2 (Pin_2)
Changed lines of the file:
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@@
-	(wire
-		(pts
-			(xy 144.78 160.02) (xy 142.24 160.02)
-		)
-		(stroke
-			(width 0)
-			(type default)
-		)
-	)
 	(wire
 		(pts
@@
 	(wire
 		(pts
+			(xy 177.8 130.81) (xy 182.88 130.81)
+		)
+		(stroke
+			(width 0)
+			(type default)
+		)
+	)
+	(wire
+		(pts
 			(xy 160.02 107.95) (xy 144.78 107.95)
 		)
@@
 	(wire
 		(pts
+			(xy 109.22 162.56) (xy 116.84 162.56)
+		)
+		(stroke
+			(width 0)
+			(type default)
+		)
+	)
+	(wire
+		(pts
 			(xy 59.69 153.67) (xy 59.69 156.21)
 		)
@@
 	(wire
 		(pts
+			(xy 109.22 127) (xy 109.22 162.56)
+		)
+		(stroke
+			(width 0)
+			(type default)
+		)
+	)
+	(wire
+		(pts
 			(xy 109.22 127) (xy 144.78 127)
 		)
@@
 	(wire
 		(pts
-			(xy 144.78 156.21) (xy 144.78 160.02)
+			(xy 144.78 156.21) (xy 144.78 162.56)
+		)
+		(stroke
+			(width 0)
+			(type default)
+		)
+	)
+	(wire
+		(pts
+			(xy 144.78 162.56) (xy 142.24 162.56)
 		)
 		(stroke
@@
 	(wire
 		(pts
-			(xy 109.22 127) (xy 109.22 160.02)
-		)
-		(stroke
-			(width 0)
-			(type default)
-		)
-	)
-	(wire
-		(pts
 			(xy 142.24 90.17) (xy 142.24 110.49)
-		)
-		(stroke
-			(width 0)
-			(type default)
-		)
-	)
-	(wire
-		(pts
-			(xy 116.84 160.02) (xy 109.22 160.02)
 		)
 		(stroke
@@
 				(path "/9af06756-81cc-4295-8d37-80e0f168a4af"
 					(reference "J5")
+					(unit 1)
+				)
+			)
+		)
+	)
+	(symbol
+		(lib_id "Connector:Conn_01x04_Pin")
+		(at 172.72 135.89 90)
+		(unit 1)
+		(exclude_from_sim no)
+		(in_bom yes)
+		(on_board yes)
+		(dnp no)
+		(fields_autoplaced yes)
+		(property "Reference" "J2"
+			(at 173.99 138.43 90)
+			(effects
+				(font
+					(size 1.27 1.27)
+				)
+			)
+		)
+		(property "Value" "Conn_01x04_Pin"
+			(at 173.99 140.97 90)
+			(effects
+				(font
+					(size 1.27 1.27)
+				)
+			)
+		)
+		(property "Footprint" "Connector_PinHeader_2.54mm:PinHeader_1x04_P2.54mm_Vertical"
+			(at 172.72 135.89 0)
+			(effects
+				(font
+					(size 1.27 1.27)
+				)
+				(hide yes)
+			)
+		)
+		(property "Datasheet" "~"
+			(at 172.72 135.89 0)
+			(effects
+				(font
+					(size 1.27 1.27)
+				)
+				(hide yes)
+			)
+		)
+		(property "Description" "Generic connector, single row, 01x04, script generated"
+			(at 172.72 135.89 0)
+			(effects
+				(font
+					(size 1.27 1.27)
+				)
+				(hide yes)
+			)
+		)
+		(pin "2"
+		)
+		(pin "1"
+		)
+		(pin "3"
+		)
+		(pin "4"
+		)
+		(instances
+			(project ""
+				(path "/9af06756-81cc-4295-8d37-80e0f168a4af"
+					(reference "J2")
 					(unit 1)
 				)
@@
 			)
 		)
-		(property "Footprint" "Package_TO_SOT_SMD:SOT-23-5"
+		(property "Footprint" "Package_SO:TSOP-5_1.65x3.05mm_P0.95mm"
 			(at 71.12 146.05 0)
 			(effects
@@
 					(unit 1)
 				)
-			)
-		)
-	)
-	(symbol
-		(lib_id "Connector_Generic:Conn_01x06")
-		(at 177.8 135.89 270)
-		(unit 1)
-		(exclude_from_sim no)
-		(in_bom yes)
-		(on_board yes)
-		(dnp no)
-		(property "Reference" "J2"
-			(at 163.83 135.89 0)
-			(effects
-				(font
-					(size 1.27 1.27)
-				)
-			)
-		)
-		(property "Value" "RADIO"
-			(at 166.37 135.89 0)
-			(effects
-				(font
-					(size 1.27 1.27)
-				)
-			)
-		)
-		(property "Footprint" "Connector_JST:JST_SH_BM06B-SRSS-TB_1x06-1MP_P1.00mm_Vertical"
-			(at 177.8 135.89 0)
-			(effects
-				(font
-					(size 1.27 1.27)
-				)
-				(hide yes)
-			)
-		)
-		(property "Datasheet" "~"
-			(at 177.8 135.89 0)
-			(effects
-				(font
-					(size 1.27 1.27)
-				)
-				(hide yes)
-			)
-		)
-		(property "Description" "Generic connector, single row, 01x06, script generated (kicad-library-utils/schlib/autogen/connector/)"
-			(at 177.8 135.89 0)
-			(effects
-				(font
-					(size 1.27 1.27)
-				)
-				(hide yes)
-			)
-		)
-		(pin "2"
-		)
-		(pin "1"
-		)
-		(pin "4"
-		)
-		(pin "5"
-		)
-		(pin "3"
-		)
-		(pin "6"
-		)
-		(instances
-			(project ""
-				(path "/9af06756-81cc-4295-8d37-80e0f168a4af"
-					(reference "J2")
-					(unit 1)
-				)

Commit message: New PCB, progress on esp32 code
Parts:
- removed C1: 1uF_50V, Capacitor_THT:C_Disc_D5.0mm_W2.5mm_P5.00mm, symbol PCM_SL_Capacitors:1uF_50V
- removed J2: Conn_01x04_Pin, Connector_PinHeader_2.54mm:PinHeader_1x04_P2.54mm_Vertical, symbol Connector:Conn_01x04_Pin
- removed J4: 9DOF, Connector_PinHeader_2.54mm:PinHeader_1x11_P2.54mm_Vertical, symbol Connector_Generic_MountingPin:Conn_01x10_MountingPin
- removed J5: GPS, Connector_PinHeader_2.54mm:PinHeader_1x03_P2.54mm_Vertical, symbol Connector:Conn_01x03_Pin
- removed U4: SN74AVC4T245PW, Package_SO:TSSOP-16_4.4x5mm_P0.65mm, symbol Logic_LevelTranslator:SN74AVC4T245PW
- removed U5: NCP163ASN180T1G, Package_SO:TSOP-5_1.65x3.05mm_P0.95mm, symbol Regulator_Linear:NCP163ASN180T1G
- added J2: Conn_01x06, Connector_PinHeader_2.54mm:PinHeader_1x06_P2.54mm_Vertical, symbol Connector_Generic:Conn_01x06
- added J4: Conn_01x05_Pin, symbol Connector:Conn_01x05_Pin
Connections:
- net +5V: now also J2.6 (Pin_6), J4.2 (Pin_2)
- net GND: now also J2.1 (Pin_1), J4.1 (Pin_1)
- net at U3.31 (IO19): now also J4.5 (Pin_5)
- net at U3.30 (IO18): now also J2.5 (Pin_5)
- net at U3.29 (IO5): now also J2.4 (Pin_4)
- net at U3.27 (IO16): now also J2.2 (Pin_2)
- net at U3.28 (IO17): now also J2.3 (Pin_3)
- no-connect marks 0 -> 1

Commit message: Progress on esp32
Parts:
- removed J2: Conn_01x06, Connector_PinHeader_2.54mm:PinHeader_1x06_P2.54mm_Vertical, symbol Connector_Generic:Conn_01x06
- added J5: Conn_01x04_Pin, Connector_PinHeader_2.54mm:PinHeader_1x04_P2.54mm_Vertical, symbol Connector:Conn_01x04_Pin
Connections:
- net +5V: now also J5.1 (Pin_1)
- net GND: now also J5.4 (Pin_4)
- net at U3.29 (IO5): now also J5.3 (Pin_3)
- net at U3.30 (IO18): now also J5.2 (Pin_2)
Changed lines of the file:
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@@
-	(wire
-		(pts
-			(xy 154.94 100.33) (xy 154.94 90.17)
-		)
-		(stroke
-			(width 0)
-			(type default)
-		)
-	)
-	(wire
-		(pts
-			(xy 177.8 101.6) (xy 152.4 101.6)
-		)
-		(stroke
-			(width 0)
-			(type default)
-		)
-	)
 	(wire
 		(pts
@@
 	(wire
 		(pts
-			(xy 180.34 100.33) (xy 154.94 100.33)
-		)
-		(stroke
-			(width 0)
-			(type default)
-		)
-	)
-	(wire
-		(pts
 			(xy 157.48 110.49) (xy 142.24 110.49)
 		)
@@
 	(wire
 		(pts
+			(xy 177.8 130.81) (xy 182.88 130.81)
+		)
+		(stroke
+			(width 0)
+			(type default)
+		)
+	)
+	(wire
+		(pts
 			(xy 172.72 130.81) (xy 172.72 106.68)
 		)
@@
 	(wire
 		(pts
-			(xy 152.4 90.17) (xy 152.4 101.6)
-		)
-		(stroke
-			(width 0)
-			(type default)
-		)
-	)
-	(wire
-		(pts
 			(xy 170.18 130.81) (xy 170.18 123.19)
 		)
@@
 	(wire
 		(pts
-			(xy 177.8 130.81) (xy 177.8 101.6)
-		)
-		(stroke
-			(width 0)
-			(type default)
-		)
-	)
-	(wire
-		(pts
 			(xy 160.02 107.95) (xy 144.78 107.95)
 		)
@@
 		(pts
 			(xy 167.64 104.14) (xy 167.64 90.17)
-		)
-		(stroke
-			(width 0)
-			(type default)
-		)
-	)
-	(wire
-		(pts
-			(xy 180.34 130.81) (xy 180.34 100.33)
 		)
 		(stroke
@@
 	)
 	(symbol
-		(lib_id "Connector_Generic:Conn_01x06")
-		(at 177.8 135.89 270)
+		(lib_id "Connector:Conn_01x04_Pin")
+		(at 172.72 135.89 90)
 		(unit 1)
 		(exclude_from_sim no)
@@
 		(dnp no)
 		(fields_autoplaced yes)
-		(property "Reference" "J2"
-			(at 176.53 139.7 90)
-			(effects
-				(font
-					(size 1.27 1.27)
-				)
-			)
-		)
-		(property "Value" "Conn_01x06"
-			(at 176.53 142.24 90)
-			(effects
-				(font
-					(size 1.27 1.27)
-				)
-			)
-		)
-		(property "Footprint" "Connector_PinHeader_2.54mm:PinHeader_1x06_P2.54mm_Vertical"
-			(at 177.8 135.89 0)
+		(property "Reference" "J5"
+			(at 173.99 138.43 90)
+			(effects
+				(font
+					(size 1.27 1.27)
+				)
+			)
+		)
+		(property "Value" "Conn_01x04_Pin"
+			(at 173.99 140.97 90)
+			(effects
+				(font
+					(size 1.27 1.27)
+				)
+			)
+		)
+		(property "Footprint" "Connector_PinHeader_2.54mm:PinHeader_1x04_P2.54mm_Vertical"
+			(at 172.72 135.89 0)
 			(effects
 				(font
@@
 		)
 		(property "Datasheet" "~"
-			(at 177.8 135.89 0)
-			(effects
-				(font
-					(size 1.27 1.27)
-				)
-				(hide yes)
-			)
-		)
-		(property "Description" "Generic connector, single row, 01x06, script generated (kicad-library-utils/schlib/autogen/connector/)"
-			(at 177.8 135.89 0)
-			(effects
-				(font
-					(size 1.27 1.27)
-				)
-				(hide yes)
-			)
+			(at 172.72 135.89 0)
+			(effects
+				(font
+					(size 1.27 1.27)
+				)
+				(hide yes)
+			)
+		)
+		(property "Description" "Generic connector, single row, 01x04, script generated"
+			(at 172.72 135.89 0)
+			(effects
+				(font
+					(size 1.27 1.27)
+				)
+				(hide yes)
+			)
+		)
+		(pin "3"
+		)
+		(pin "4"
+		)
+		(pin "2"
 		)
 		(pin "1"
-		)
-		(pin "2"
-		)
-		(pin "5"
-		)
-		(pin "3"
-		)
-		(pin "6"
-		)
-		(pin "4"
 		)
 		(instances
 			(project ""
 				(path "/9af06756-81cc-4295-8d37-80e0f168a4af"
-					(reference "J2")
+					(reference "J5")
 					(unit 1)
 				)
